Commit message: iiwa hardware test

File: wsg50-ros-pkg/wsg_50_simulation/urdf/wsg_50.urdf.xacro (robot description, xacro)
@@ -15,5 +15,5 @@
  </joint>
 <!-- BASE LINK -->
- <link name="${name}_base_link">
+   <link name="${name}_base_link">
       <inertial>
           <mass value="0.25" />
@@ -28,5 +28,5 @@
           <geometry>
              <mesh filename="package://wsg_50_simulation/meshes/WSG50_110.stl" scale="1 1 1"/>
-	     <!--box size="0.146 0.05 0.0735"/-->
+	         <!--box size="0.146 0.05 0.0735"/-->
           </geometry>
           <material name="grey">
@@ -37,13 +37,13 @@
           <origin xyz="0.0 0 0" rpy="0 0 0" />
           <geometry>
-	     <!--box size="0.146 0.05 0.0735"/-->
-             <mesh filename="package://wsg_50_simulation/meshes/WSG50_110.stl" scale="1 1 1"/>
-         </geometry>
-     </collision>
-  </link>
-  <gazebo reference="${name}_base_link">
-    <material>Gazebo/Grey</material>
-    <turnGravityOff>false</turnGravityOff>
-  </gazebo>
+	         <!--box size="0.146 0.05 0.0735"/-->
+            <mesh filename="package://wsg_50_simulation/meshes/WSG50_110.stl" scale="1 1 1"/>
+         </geometry>
+     </collision>
+   </link>
+   <gazebo reference="${name}_base_link">
+      <material>Gazebo/Grey</material>
+      <turnGravityOff>false</turnGravityOff>
+   </gazebo>
   <joint name="${name}_center_joint" type="fixed">
      <origin xyz="0 0 ${finger_length}" rpy="0 0 0" />      <!--origin xyz="-0.0067 0 0.049" rpy="0 0 0" /-->
@@ -83,81 +83,81 @@
   <link name="${name}_gripper_left">
       <inertial>
-          <mass value="0.1" />
-          <origin xyz="0 0 0" />
-      <inertia ixx="1.0" ixy="0.0" ixz="0.0"
-               iyy="1.0" iyz="0.0"
-               izz="1.0" />
-      </inertial>
-      <visual>
-          <origin xyz="0.0 0 0" rpy="0 0 0" />
-          <geometry>
-             <mesh filename="package://wsg_50_simulation/meshes/GUIDE_WSG50_110.stl" scale="0.001 0.001 0.001"/>
-	     <!--box size="0.0175 0.03 0.024"/-->
-          </geometry>
-          <material name="black">
-		<color rgba="0 0 0 0"/>
-      	  </material>
-      </visual>
-      <collision>
-          <origin xyz="0 0 0" rpy="0 0 0" />
-          <geometry>
-	     <!--box size="0.0175 0.03 0.024"/-->
-             <mesh filename="package://wsg_50_simulation/meshes/GUIDE_WSG50_110.stl" scale="0.001 0.001 0.001"/>
-         </geometry>
-     </collision>
-     <contact_coefficients kd="1.0" kp="1000.0" mu="0"/>
-  </link>
-  <gazebo reference="${name}_gripper_left">
-    <material>Gazebo/Blue</material>
-    <turnGravityOff>false</turnGravityOff>
-  </gazebo>
-  <!-- LEFT FINGER -->
-  <joint name="${name}_guide_joint_finger_left" type="fixed">
-     <origin xyz="${finger_tip} 0 ${finger_length}" rpy="0 0 0" />
-     <parent link="${name}_gripper_left"/>
-     <child link="${name}_finger_left" />
-     <dynamics friction="100" damping="100" />
-     <axis xyz="1 0 0"/>
-     <limit effort="100" velocity="100"/>
-  </joint>
+         <mass value="0.1" />
+         <origin xyz="0 0 0" />
+         <inertia ixx="1.0" ixy="0.0" ixz="0.0"
+               iyy="1.0" iyz="0.0"
+               izz="1.0" />
+      </inertial>
+      <visual>
+         <origin xyz="0.0 0 0" rpy="0 0 0" />
+         <geometry>
+            <mesh filename="package://wsg_50_simulation/meshes/GUIDE_WSG50_110.stl" scale="0.001 0.001 0.001"/>
+            <!--box size="0.0175 0.03 0.024"/-->
+         </geometry>
+         <material name="black">
+	         <color rgba="0 0 0 0"/>
+         </material>
+      </visual>
+      <collision>
+         <origin xyz="0 0 0" rpy="0 0 0" />
+         <geometry>
+	         <!--box size="0.0175 0.03 0.024"/-->
+            <mesh filename="package://wsg_50_simulation/meshes/GUIDE_WSG50_110.stl" scale="0.001 0.001 0.001"/>
+         </geometry>
+     </collision>
+     <contact_coefficients kd="1.0" kp="1000.0" mu="0"/>
+   </link>
+   <gazebo reference="${name}_gripper_left">
+      <material>Gazebo/Blue</material>
+      <turnGravityOff>false</turnGravityOff>
+   </gazebo>
+   <!-- LEFT FINGER -->
+   <joint name="${name}_guide_joint_finger_left" type="fixed">
+      <origin xyz="${finger_tip} 0 ${finger_length}" rpy="0 0 0" />
+      <parent link="${name}_gripper_left"/>
+      <child link="${name}_finger_left" />
+      <dynamics friction="100" damping="100" />
+      <axis xyz="1 0 0"/>
+      <limit effort="100" velocity="100"/>
+   </joint>
   <link name="${name}_finger_left">
       <inertial>
-          <mass value="0.1" />
-          <origin xyz="0 0 0" />
-      <inertia ixx="1.0" ixy="0.0" ixz="0.0"
-               iyy="1.0" iyz="0.0"
-               izz="1.0" />
-      </inertial>
-      <visual>
-          <origin xyz="0.0 0 0" rpy="0 0 0" />
-          <geometry>
-             <mesh filename="package://wsg_50_simulation/meshes/WSG-FMF.stl" scale="0.001 0.001 0.001"/>
-          </geometry>
-          <material name="black">
-		<color rgba="0 0 0 0"/>
-      	  </material>
-      </visual>
-      <collision>
-          <origin xyz="0 0 0" rpy="0 0 0" />
-          <geometry>
-             <mesh filename="package://wsg_50_simulation/meshes/WSG-FMF.stl" scale="0.001 0.001 0.001"/>
-         </geometry>
-     </collision>
-     <contact_coefficients kd="1.0" kp="1000.0" mu="0"/>
-  </link>
-  <gazebo reference="${name}_finger_left">
-    <material>Gazebo/Blue</material>
-    <turnGravityOff>false</turnGravityOff>
-  </gazebo>
+         <mass value="0.1" />
+         <origin xyz="0 0 0" />
+         <inertia ixx="1.0" ixy="0.0" ixz="0.0"
+               iyy="1.0" iyz="0.0"
+               izz="1.0" />
+      </inertial>
+      <visual>
+         <origin xyz="0.0 0 0" rpy="0 0 0" />
+         <geometry>
+            <mesh filename="package://wsg_50_simulation/meshes/WSG-FMF.stl" scale="0.001 0.001 0.001"/>
+         </geometry>
+         <material name="black">
+		      <color rgba="0 0 0 0"/>
+      	</material>
+      </visual>
+      <collision>
+         <origin xyz="0 0 0" rpy="0 0 0" />
+         <geometry>
+            <mesh filename="package://wsg_50_simulation/meshes/WSG-FMF.stl" scale="0.001 0.001 0.001"/>
+         </geometry>
+     </collision>
+     <contact_coefficients kd="1.0" kp="1000.0" mu="0"/>
+  </link>
+   <gazebo reference="${name}_finger_left">
+      <material>Gazebo/Blue</material>
+      <turnGravityOff>false</turnGravityOff>
+   </gazebo>
   <!-- GRIPPER RIGHT -->
   <joint name="${name}_finger_right_joint" type="prismatic">
-     <limit lower="0.0027" upper="0.055" effort="1.0" velocity="1.0"/>
-     <origin xyz="0 0 0" rpy="0 0 3.14159" />
-     <parent link="${name}_base_link"/>
-     <child link="${name}_gripper_right" />
-     <axis xyz="-1 0 0"/>
-     <dynamics friction="100" damping="100" />
-     <limit effort="100" velocity="100"/>
-  </joint>
+      <limit lower="0.0027" upper="0.055" effort="1.0" velocity="1.0"/>
+      <origin xyz="0 0 0" rpy="0 0 3.14159" />
+      <parent link="${name}_base_link"/>
+      <child link="${name}_gripper_right" />
+      <axis xyz="-1 0 0"/>
+      <dynamics friction="100" damping="100" />
+      <limit effort="100" velocity="100"/>
+   </joint>
   <!--transmission name="${name}_base_trans_right" type="pr2_mechanism_model/SimpleTransmission">
      <actuator name="${name}_base_motor_right" />
@@ -167,19 +167,19 @@
      <hardwareInterface>hardware_interface/EffortJointInterface</hardwareInterface>
   </transmission-->
-  <transmission name="${name}_base_trans_left">
-     <type>transmission_interface/SimpleTransmission</type>
-     <actuator name="${name}_base_motor_left">
-       <hardwareInterface>hardware_interface/EffortJointInterface</hardwareInterface>
-       <mechanicalReduction>1</mechanicalReduction>
-       <!--motorTorqueConstant>1</motorTorqueConstant-->
-     </actuator>
-     <joint name="${name}_finger_right_joint">
-      <hardwareInterface>hardware_interface/EffortJointInterface</hardwareInterface>
-     </joint>
-  </transmission>
-    <link name="${name}_gripper_right">
-      <inertial>
-          <mass value="0.1" />
-          <origin xyz="0 0 0" />
+   <transmission name="${name}_base_trans_left">
+      <type>transmission_interface/SimpleTransmission</type>
+      <actuator name="${name}_base_motor_left">
+         <hardwareInterface>hardware_interface/EffortJointInterface</hardwareInterface>
+         <mechanicalReduction>1</mechanicalReduction>
+         <!--motorTorqueConstant>1</motorTorqueConstant-->
+      </actuator>
+      <joint name="${name}_finger_right_joint">
+         <hardwareInterface>hardware_interface/EffortJointInterface</hardwareInterface>
+      </joint>
+   </transmission>
+   <link name="${name}_gripper_right">
+      <inertial>
+         <mass value="0.1" />
+         <origin xyz="0 0 0" />
       <inertia ixx="1.0" ixy="0.0" ixz="0.0"
                iyy="1.0" iyz="0.0"
@@ -187,18 +187,18 @@
       </inertial>
       <visual>
-          <origin xyz="0.0 0 0" rpy="0 0 0" />
-          <geometry>
-             <mesh filename="package://wsg_50_simulation/meshes/GUIDE_WSG50_110.stl" scale="0.001 0.001 0.001"/>
-	     <!--box size="0.0175 0.03 0.024"/-->
-          </geometry>
-          <material name="black">
-		<color rgba="0 0 0 0"/>
-      	  </material>
-      </visual>
-      <collision>
-          <origin xyz="0 0 0" rpy="0 0 0" />
-          <geometry>
-	     <!--box size="0.0175 0.03 0.024"/-->
-             <mesh filename="package://wsg_50_simulation/meshes/GUIDE_WSG50_110.stl" scale="0.001 0.001 0.001"/>
+         <origin xyz="0.0 0 0" rpy="0 0 0" />
+         <geometry>
+            <mesh filename="package://wsg_50_simulation/meshes/GUIDE_WSG50_110.stl" scale="0.001 0.001 0.001"/>
+	         <!--box size="0.0175 0.03 0.024"/-->
+         </geometry>
+         <material name="black">
+		      <color rgba="0 0 0 0"/>
+      	</material>
+      </visual>
+      <collision>
+         <origin xyz="0 0 0" rpy="0 0 0" />
+         <geometry>
+	         <!--box size="0.0175 0.03 0.024"/-->
+            <mesh filename="package://wsg_50_simulation/meshes/GUIDE_WSG50_110.stl" scale="0.001 0.001 0.001"/>
          </geometry>
      </collision>
@@ -220,6 +220,6 @@
   <link name="${name}_finger_right">
       <inertial>
-          <mass value="0.1" />
-          <origin xyz="0 0 0" />
+         <mass value="0.1" />
+         <origin xyz="0 0 0" />
       <inertia ixx="1.0" ixy="0.0" ixz="0.0"
                iyy="1.0" iyz="0.0"
@@ -227,16 +227,16 @@
       </inertial>
       <visual>
-          <origin xyz="0.0 0 0" rpy="0 0 0" />
-          <geometry>
-             <mesh filename="package://wsg_50_simulation/meshes/WSG-FMF.stl" scale="0.001 0.001 0.001"/>
-          </geometry>
-          <material name="black">
-		<color rgba="0 0 0 0"/>
-      	  </material>
-      </visual>
-      <collision>
-          <origin xyz="0 0 0" rpy="0 0 0" />
-          <geometry>
-             <mesh filename="package://wsg_50_simulation/meshes/WSG-FMF.stl" scale="0.001 0.001 0.001"/>
+         <origin xyz="0.0 0 0" rpy="0 0 0" />
+         <geometry>
+            <mesh filename="package://wsg_50_simulation/meshes/WSG-FMF.stl" scale="0.001 0.001 0.001"/>
+         </geometry>
+         <material name="black">
+		      <color rgba="0 0 0 0"/>
+      	</material>
+      </visual>
+      <collision>
+         <origin xyz="0 0 0" rpy="0 0 0" />
+         <geometry>
+            <mesh filename="package://wsg_50_simulation/meshes/WSG-FMF.stl" scale="0.001 0.001 0.001"/>
          </geometry>
      </collision>
